File: mic_boards/mic_boards.kicad_pcb (KiCad board)
At the start: 4 copper layers, 258 x 325 mm, 114 parts, among them J1 Test Points, U1 SN74LVC2G17DBVR, U26 10056847-101LF

Commit message: Redo layout (wip)
Parts:
- removed REF**1: MountingHole_3.2mm_M3_DIN965, MountingHole:MountingHole_3.2mm_M3_DIN965
- moved REF**10 2.00 mm to (248.0, 205.0)
- moved REF**4 2.00 mm to (248.0, 10.0)
- moved REF**7 2.00 mm to (248.0, 100.0)
Routing:
- net +3V3: track 277.6 -> 278.1 mm
Other:
- outline, holes or cut-outs redrawn
Changed lines of the file:
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@@
 	(footprint "MountingHole:MountingHole_3.2mm_M3_DIN965"
 		(layer "F.Cu")
-		(at 250 205)
+		(at 248 205)
 		(descr "Mounting Hole 3.2mm, M3, no annular, generated by kicad-footprint-generator mountinghole.py")
 		(tags "mountinghole M3 DIN965")
@@
 	(footprint "MountingHole:MountingHole_3.2mm_M3_DIN965"
 		(layer "F.Cu")
-		(at 250 100)
+		(at 248 100)
 		(descr "Mounting Hole 3.2mm, M3, no annular, generated by kicad-footprint-generator mountinghole.py")
 		(tags "mountinghole M3 DIN965")
@@
 	(footprint "MountingHole:MountingHole_3.2mm_M3_DIN965"
 		(layer "F.Cu")
-		(at 250 10)
+		(at 248 10)
 		(descr "Mounting Hole 3.2mm, M3, no annular, generated by kicad-footprint-generator mountinghole.py")
 		(tags "mountinghole M3 DIN965")
@@
 	(footprint "MountingHole:MountingHole_3.2mm_M3_DIN965"
 		(layer "F.Cu")
-		(at 250 315)
-		(descr "Mounting Hole 3.2mm, M3, no annular, generated by kicad-footprint-generator mountinghole.py")
-		(tags "mountinghole M3 DIN965")
-		(property "Reference" "REF**1"
-			(at 0 -3.75 0)
-			(layer "F.SilkS")
-			(hide yes)
-			(effects
-				(font
-					(size 1 1)
-					(thickness 0.15)
-				)
-			)
-		)
-		(property "Value" "MountingHole_3.2mm_M3_DIN965"
-			(at 0 3.75 0)
-			(layer "F.Fab")
-			(effects
-				(font
-					(size 1 1)
-					(thickness 0.15)
-				)
-			)
-		)
-		(property "Datasheet" ""
-			(at 0 0 0)
-			(layer "F.Fab")
-			(hide yes)
-			(effects
-				(font
-					(size 1.27 1.27)
-					(thickness 0.15)
-				)
-			)
-		)
-		(property "Description" ""
-			(at 0 0 0)
-			(layer "F.Fab")
-			(hide yes)
-			(effects
-				(font
-					(size 1.27 1.27)
-					(thickness 0.15)
-				)
-			)
-		)
-		(attr exclude_from_pos_files exclude_from_bom)
-		(fp_circle
-			(center 0 0)
-			(end 2.8 0)
-			(stroke
-				(width 0.15)
-				(type solid)
-			)
-			(fill no)
-			(layer "Cmts.User")
-		)
-		(fp_circle
-			(center 0 0)
-			(end 3.05 0)
-			(stroke
-				(width 0.05)
-				(type solid)
-			)
-			(fill no)
-			(layer "F.CrtYd")
-		)
-		(fp_text user "${REFERENCE}"
-			(at 0 0 0)
-			(layer "F.Fab")
-			(effects
-				(font
-					(size 1 1)
-					(thickness 0.15)
-				)
-			)
-		)
-		(pad "" np_thru_hole circle
-			(at 0 0)
-			(size 3.2 3.2)
-			(drill 3.2)
-			(layers "*.Cu" "*.Mask")
-		)
-		(embedded_fonts no)
-	)
-	(footprint "MountingHole:MountingHole_3.2mm_M3_DIN965"
-		(layer "F.Cu")
 		(at 135 205)
 		(descr "Mounting Hole 3.2mm, M3, no annular, generated by kicad-footprint-generator mountinghole.py")
@@
 	)
 	(gr_line
-		(start 258 325)
-		(end 258 0)
+		(start 258.004065 201.995935)
+		(end 258.00004 1.99996)
 		(stroke
 			(width 0.05)
@@
 	(gr_line
 		(start 11 13)
-		(end 11 325)
+		(end 11 323)
 		(stroke
 			(width 0.05)
@@
 		(layer "Edge.Cuts")
 	)
+	(gr_arc
+		(start 256.00004 0)
+		(mid 257.414239 0.585772)
+		(end 258.00004 1.99996)
+		(stroke
+			(width 0.05)
+			(type default)
+		)
+		(layer "Edge.Cuts")
+	)
+	(gr_arc
+		(start 13 325)
+		(mid 11.585786 324.414214)
+		(end 11 323)
+		(stroke
+			(width 0.05)
+			(type default)
+		)
+		(layer "Edge.Cuts")
+	)
+	(gr_arc
+		(start 0 1)
+		(mid 0.292893 0.292893)
+		(end 1 0)
+		(stroke
+			(width 0.05)
+			(type default)
+		)
+		(layer "Edge.Cuts")
+	)
+	(gr_arc
+		(start 1 13)
+		(mid 0.292893 12.707107)
+		(end 0 12)
+		(stroke
+			(width 0.05)
+			(type default)
+		)
+		(layer "Edge.Cuts")
+	)
 	(gr_line
-		(start 0 0)
-		(end 0 13)
+		(start 0 1)
+		(end 0 12)
+		(stroke
+			(width 0.05)
+			(type default)
+		)
+		(layer "Edge.Cuts")
+	)
+	(gr_arc
+		(start 258.004065 201.995935)
+		(mid 221.977008 288.972943)
+		(end 135 325)
 		(stroke
 			(width 0.05)
@@
 	)
 	(gr_line
-		(start 11 325)
-		(end 258 325)
+		(start 13 325)
+		(end 135 325)
 		(stroke
 			(width 0.05)
@@
 	)
 	(gr_line
-		(start 0 13)
+		(start 1 13)
 		(end 11 13)
 		(stroke
@@
 	)
 	(gr_line
-		(start 258 0)
-		(end 0 0)
+		(start 256.00004 0)
+		(end 1 0)
 		(stroke
 			(width 0.05)
@@
 	(via
 		(at 12.1 9.9)
-		(size 0.6)
-		(drill 0.3)
+		(size 0.8)
+		(drill 0.4)
 		(layers "F.Cu" "B.Cu")
 		(free yes)
@@
 	(segment
 		(start 10.1 2.7)
-		(end 11.7 2.7)
+		(end 12.2 2.7)
 		(width 0.3)
 		(layer "F.Cu")
@@
 	)
 	(via
-		(at 11.7 2.7)
-		(size 0.6)
-		(drill 0.3)
+		(at 12.2 2.7)
+		(size 0.8)
+		(drill 0.4)
 		(layers "F.Cu" "B.Cu")
 		(free yes)
